Commit message: Added pick-and-place implementation for Step4

File: Step4/ur3e_on_table.urdf.xacro (robot description, xacro)
@@ -1,8 +1,11 @@
 <?xml version="1.0" encoding="UTF-8"?>
-<robot xmlns:xacro="http://wiki.ros.org/xacro" name="table">
-    <xacro:include filename="$(find table_description)/urdf/materials.xacro" />
-    <xacro:include filename="$(find table_description)/urdf/table_macro.xacro" />
+<robot xmlns:xacro="http://www.ros.org/wiki/xacro" name="ur3e_on_table">
+    <!-- Use LOCAL includes inside this package -->
+    <xacro:include filename="materials.xacro" />
+    <xacro:include filename="table_macro.xacro" />
     <link name="world" />
+    <!-- Table -->
     <xacro:table prefix="table_" parent="world">
+        <!-- table position in the world -->
         <origin xyz="0 0 1" rpy="0 0 0" />
     </xacro:table>
@@ -13,5 +16,4 @@
     <!-- possible 'ur_type' values: ur3, ur3e, ur5, ur5e, ur7e, ur10, ur10e, ur12e, ur16e, ur15,
     ur20, ur30 -->
-    <!-- the default value should raise an error in case this was called without defining the type -->
     <xacro:arg name="ur_type" default="ur3e" />
     <!-- parameters -->
@@ -29,5 +31,5 @@
     <xacro:arg name="safety_pos_margin" default="0.15" />
     <xacro:arg name="safety_k_position" default="20" />
-    <!-- arm -->
+    <!-- arm mounted to the table top -->
     <xacro:ur_robot
         name="$(arg name)"
@@ -42,5 +44,6 @@
         safety_k_position="$(arg safety_k_position)"
     >
-        <origin xyz="0 0 0" rpy="0 0 0" />          <!-- position robot in the world -->
+        <!-- pose of robot relative to its parent link (table_top) -->
+        <origin xyz="0 0 0" rpy="0 0 0" />
     </xacro:ur_robot>
 </robot>
